File: STM32Board.kicad_sch (KiCad schematic)
At the start: 28 parts, among them J1 Conn_01x03_Male, J2 Conn_01x03_Male, J3 Conn_01x06_Male, J4 Conn_01x04_Male, J7 Conn_01x02_Male, J8 USB4105-GF-A, J9 USB4105-GF-A, SW1 SW_Push, SW2 SW_DIP_x01, U1 STM32F103C8Tx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

Commit message: add gitignore file and repair error in schematics
Parts:
- removed C1, C2, C3, C4, C9: 0.1uF, Capacitor_SMD:C_0603_1608Metric, symbol Device:CP1_Small
- removed C5: 10u, Capacitor_SMD:C_0603_1608Metric, symbol Device:CP1_Small
- removed C6: 22u, Capacitor_Tantalum_SMD:CP_EIA-3216-18_Kemet-A, symbol Device:CP1_Small
- added C1, C2, C3, C4, C5: 0.1uF, Capacitor_SMD:C_0603_1608Metric, symbol Device:C
- added C6: 22uF, Capacitor_Tantalum_SMD:CP_EIA-3216-18_Kemet-A, symbol Device:C
- added C9: 10uF, Capacitor_SMD:C_0603_1608Metric, symbol Device:C
- U2: footprint Package_TO_SOT_SMD:SOT-223 -> Package_TO_SOT_SMD:SOT-223-3_TabPin2
Connections:
- net +3V3: now also C2.2, C3.2, C4.2, C5.2, C6.1
- net +5V: now also C9.1
- net GND: now also C1.2, C2.1, C3.1, C4.1, C5.1, C6.2, C9.2
- net at R1.1, SW1.1, U1.7 (NRST): now also C1.1
- net at J8.A4_B9 (VBUS): no longer J8.B4_A9 (VBUS)
- no-connect marks 13 -> 38
Other:
- moved on the sheet: R4, R5, R6

Commit message: Add gerber file, change the 3.3 and gnd def
Parts:
- removed SW2: SW_DIP_x01, Button_Switch_THT:SW_Slide_1P2T_CK_OS102011MS2Q, symbol Switch:SW_DIP_x01
- added SW?: SW_SPDT, Button_Switch_THT:SW_Slide_1P2T_CK_OS102011MS2Q, symbol Switch:SW_SPDT
Connections:
- net +3V3: now also J4.4 (Pin_4); no longer J4.3 (Pin_3)
- net +5V: now also SW?.2 (B)
- net GND: now also J4.3 (Pin_3), SW?.4 (SH1), SW?.5 (SH1); no longer J4.4 (Pin_4)
- net VBUS: now also SW?.1 (A)
Changed lines of the file:
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@@
   (junction (at 78.74 25.4) (diameter 0) (color 0 0 0 0)
+  )
+  (junction (at 251.46 109.22) (diameter 0) (color 0 0 0 0)
   )
   (junction (at 242.57 120.65) (diameter 0) (color 0 0 0 0)
@@
     (stroke (width 0) (type default) (color 0 0 0 0))
   )
+  (wire (pts (xy 251.46 109.22) (xy 251.46 104.14))
+    (stroke (width 0) (type default) (color 0 0 0 0))
+  )
   (wire (pts (xy 58.42 26.67) (xy 60.96 26.67))
     (stroke (width 0) (type default) (color 0 0 0 0))
@@
     (stroke (width 0) (type default) (color 0 0 0 0))
   )
+  (wire (pts (xy 255.27 111.76) (xy 255.27 109.22))
+    (stroke (width 0) (type default) (color 0 0 0 0))
+  )
   (wire (pts (xy 137.16 31.75) (xy 137.16 33.02))
     (stroke (width 0) (type default) (color 0 0 0 0))
@@
     (stroke (width 0) (type default) (color 0 0 0 0))
   )
+  (wire (pts (xy 251.46 111.76) (xy 251.46 109.22))
+    (stroke (width 0) (type default) (color 0 0 0 0))
+  )
   (wire (pts (xy 168.91 148.59) (xy 166.37 148.59))
     (stroke (width 0) (type default) (color 0 0 0 0))
   )
   (wire (pts (xy 113.03 33.02) (xy 113.03 31.75))
+    (stroke (width 0) (type default) (color 0 0 0 0))
+  )
+  (wire (pts (xy 255.27 109.22) (xy 251.46 109.22))
     (stroke (width 0) (type default) (color 0 0 0 0))
   )
@@
     (pin "1")
   )
-  (symbol (lib_id "power:+3.3V") (at 97.79 90.17 90) (unit 1)
-    (in_bom yes) (on_board yes)
-    (property "Reference" "#PWR0115" (id 0) (at 101.6 90.17 0)
-      (effects (font (size 1.27 1.27)) hide)
-    )
-    (property "Value" "+3.3V" (id 1) (at 92.71 90.17 0))
-    (property "Footprint" "" (id 2) (at 97.79 90.17 0)
-      (effects (font (size 1.27 1.27)) hide)
-    )
-    (property "Datasheet" "" (id 3) (at 97.79 90.17 0)
-      (effects (font (size 1.27 1.27)) hide)
-    )
-    (pin "1")
-  )
   (symbol (lib_id "Connector:Conn_01x04_Male") (at 102.87 92.71 180) (unit 1)
     (in_bom yes) (on_board yes)
@@
     )
     (property "Datasheet" "~" (id 3) (at 21.59 87.63 0)
-      (effects (font (size 1.27 1.27)) hide)
-    )
-    (pin "1")
-    (pin "2")
-  )
-  (symbol (lib_id "Switch:SW_DIP_x01") (at 254 120.65 0) (unit 1)
-    (in_bom yes) (on_board yes) (fields_autoplaced)
-    (property "Reference" "SW2" (id 0) (at 254 113.03 0))
-    (property "Value" "SW_DIP_x01" (id 1) (at 254 115.57 0))
-    (property "Footprint" "Button_Switch_THT:SW_Slide_1P2T_CK_OS102011MS2Q" (id 2) (at 254 120.65 0)
-      (effects (font (size 1.27 1.27)) hide)
-    )
-    (property "Datasheet" "~" (id 3) (at 254 120.65 0)
       (effects (font (size 1.27 1.27)) hide)
     )
@@
     (pin "1")
   )
-  (symbol (lib_id "power:GND") (at 97.79 87.63 270) (unit 1)
-    (in_bom yes) (on_board yes)
-    (property "Reference" "#PWR0116" (id 0) (at 91.44 87.63 0)
-      (effects (font (size 1.27 1.27)) hide)
-    )
-    (property "Value" "GND" (id 1) (at 93.98 83.82 0))
+  (symbol (lib_id "power:+3.3V") (at 97.79 87.63 90) (unit 1)
+    (in_bom yes) (on_board yes)
+    (property "Reference" "#PWR0102" (id 0) (at 101.6 87.63 0)
+      (effects (font (size 1.27 1.27)) hide)
+    )
+    (property "Value" "+3.3V" (id 1) (at 97.79 83.82 90))
     (property "Footprint" "" (id 2) (at 97.79 87.63 0)
       (effects (font (size 1.27 1.27)) hide)
@@
     (pin "1")
   )
+  (symbol (lib_id "power:GND") (at 97.79 90.17 270) (unit 1)
+    (in_bom yes) (on_board yes)
+    (property "Reference" "#PWR0110" (id 0) (at 91.44 90.17 0)
+      (effects (font (size 1.27 1.27)) hide)
+    )
+    (property "Value" "GND" (id 1) (at 93.98 86.36 0))
+    (property "Footprint" "" (id 2) (at 97.79 90.17 0)
+      (effects (font (size 1.27 1.27)) hide)
+    )
+    (property "Datasheet" "" (id 3) (at 97.79 90.17 0)
+      (effects (font (size 1.27 1.27)) hide)
+    )
+    (pin "1")
+  )
   (symbol (lib_id "power:+3.3V") (at 127 116.84 0) (unit 1)
     (in_bom yes) (on_board yes)
@@
     )
     (pin "1")
+  )
+  (symbol (lib_id "Switch:SW_SPDT") (at 251.46 118.11 180) (unit 1)
+    (in_bom yes) (on_board yes) (fields_autoplaced)
+    (property "Reference" "SW?" (id 0) (at 252.095 123.19 0))
+    (property "Value" "SW_SPDT" (id 1) (at 252.095 125.73 0))
+    (property "Footprint" "Button_Switch_THT:SW_Slide_1P2T_CK_OS102011MS2Q" (id 2) (at 251.46 118.11 0)
+      (effects (font (size 1.27 1.27)) hide)
+    )
+    (property "Datasheet" "~" (id 3) (at 251.46 118.11 0)
+      (effects (font (size 1.27 1.27)) hide)
+    )
+    (pin "1")
+    (pin "2")
+    (pin "3")
+    (pin "4")
+    (pin "5")
   )
   (symbol (lib_id "power:GND") (at 176.53 38.1 0) (unit 1)
@@
     (pin "1")
   )
-  (symbol (lib_id "power:+5V") (at 261.62 120.65 270) (unit 1)
-    (in_bom yes) (on_board yes) (fields_autoplaced)
-    (property "Reference" "#PWR0108" (id 0) (at 257.81 120.65 0)
-      (effects (font (size 1.27 1.27)) hide)
-    )
-    (property "Value" "+5V" (id 1) (at 265.43 120.6499 90)
-      (effects (font (size 1.27 1.27)) (justify left))
-    )
-    (property "Footprint" "" (id 2) (at 261.62 120.65 0)
-      (effects (font (size 1.27 1.27)) hide)
-    )
-    (property "Datasheet" "" (id 3) (at 261.62 120.65 0)
-      (effects (font (size 1.27 1.27)) hide)
-    )
-    (pin "1")
-  )
   (symbol (lib_id "power:GND") (at 53.34 110.49 0) (unit 1)
     (in_bom yes) (on_board yes) (fields_autoplaced)
@@
     )
     (property "Datasheet" "" (id 3) (at 53.34 110.49 0)
+      (effects (font (size 1.27 1.27)) hide)
+    )
+    (pin "1")
+  )
+  (symbol (lib_id "power:GND") (at 251.46 104.14 180) (unit 1)
+    (in_bom yes) (on_board yes)
+    (property "Reference" "#PWR?" (id 0) (at 251.46 97.79 0)
+      (effects (font (size 1.27 1.27)) hide)
+    )
+    (property "Value" "GND" (id 1) (at 247.65 102.87 0))
+    (property "Footprint" "" (id 2) (at 251.46 104.14 0)
+      (effects (font (size 1.27 1.27)) hide)
+    )
+    (property "Datasheet" "" (id 3) (at 251.46 104.14 0)
       (effects (font (size 1.27 1.27)) hide)
     )
@@
     (pin "2")
   )
+  (symbol (lib_id "power:+5V") (at 256.54 118.11 270) (unit 1)
+    (in_bom yes) (on_board yes) (fields_autoplaced)
+    (property "Reference" "#PWR?" (id 0) (at 252.73 118.11 0)
+      (effects (font (size 1.27 1.27)) hide)
+    )
+    (property "Value" "+5V" (id 1) (at 260.35 118.1099 90)
+      (effects (font (size 1.27 1.27)) (justify left))
+    )
+    (property "Footprint" "" (id 2) (at 256.54 118.11 0)
+      (effects (font (size 1.27 1.27)) hide)
+    )
+    (property "Datasheet" "" (id 3) (at 256.54 118.11 0)
+      (effects (font (size 1.27 1.27)) hide)
+    )
+    (pin "1")
+  )
   (sheet_instances
     (path "/" (page "1"))
@@
       (reference "#PWR0101") (unit 1) (value "+3.3V") (footprint "")
     )
+    (path "/37ba04c2-b201-4f29-919c-bcd861d42582"
+      (reference "#PWR0102") (unit 1) (value "+3.3V") (footprint "")
+    )
     (path "/8257417e-3db1-4b7e-a79b-84d4ba8c4011"
       (reference "#PWR0103") (unit 1) (value "GND") (footprint "")
@@
       (reference "#PWR0107") (unit 1) (value "GND") (footprint "")
     )
-    (path "/b67dfcd9-582c-42ad-bc82-5f861f85492f"
-      (reference "#PWR0108") (unit 1) (value "+5V") (footprint "")
-    )
     (path "/2f86a7e4-5198-44a2-ade0-2f6765ecdfb0"
       (reference "#PWR0109") (unit 1) (value "GND") (footprint "")
     )
+    (path "/93c82e94-97e2-43d8-ba73-ac784d4bd46a"
+      (reference "#PWR0110") (unit 1) (value "GND") (footprint "")
+    )
     (path "/1cb04a09-2170-4553-aa97-cddc7ca5b52d"
       (reference "#PWR0111") (unit 1) (value "+3.3V") (footprint "")
@@
       (reference "#PWR0114") (unit 1) (value "GND") (footprint "")
     )
-    (path "/0bd0a832-b0e1-43ea-86ff-02f01787a42f"
-      (reference "#PWR0115") (unit 1) (value "+3.3V") (footprint "")
-    )
-    (path "/41535fbb-fac6-4207-a5fb-0ce65c02f2f6"
-      (reference "#PWR0116") (unit 1) (value "GND") (footprint "")
-    )
     (path "/14eb649f-6533-4cef-8ccc-94a1fdfaa111"
       (reference "#PWR0117") (unit 1) (value "GND") (footprint "")
@@
       (reference "#PWR0130") (unit 1) (value "GND") (footprint "")
     )
+    (path "/bd62a603-dbed-4974-931f-31dce0682241"
+      (reference "#PWR?") (unit 1) (value "GND") (footprint "")
+    )
+    (path "/fe1d5bd2-f6e6-4c0c-9208-77f1349159bd"
+      (reference "#PWR?") (unit 1) (value "+5V") (footprint "")
+    )
     (path "/038b10e3-303b-49e0-9d44-1286d4150616"
       (reference "C1") (unit 1) (value "0.1uF") (footprint "Capacitor_SMD:C_0603_1608Metric")
@@
       (reference "SW1") (unit 1) (value "SW_Push") (footprint "Button_Switch_SMD:SW_Push_SPST_NO_Alps_SKRK")
     )
-    (path "/190e5db4-2e78-4247-8e9e-f143f5a2a297"
-      (reference "SW2") (unit 1) (value "SW_DIP_x01") (footprint "Button_Switch_THT:SW_Slide_1P2T_CK_OS102011MS2Q")
+    (path "/948c9332-69b9-4baf-8d8a-c76ec1388a8e"
+      (reference "SW?") (unit 1) (value "SW_SPDT") (footprint "Button_Switch_THT:SW_Slide_1P2T_CK_OS102011MS2Q")
     )
     (path "/bfb630e3-509a-4343-86ca-b017c6eec725"
